File: hardware/pcb design files/quadraptor/quadraptor.kicad_pcb (KiCad board)
At the start: 2 copper layers, 96.6 x 99.9 mm, 144 parts, among them J1 Conn_01x04, J10 Conn_01x04, J11 Conn_02x09_Odd_Even, J12 Conn_02x04, J13 Conn_01x04, J14 Conn_01x02, J15 Conn_01x02, J16 Conn_01x02, J17 Conn_01x02, J18 Conn_01x02, J19 Conn_01x04, J2 Conn_01x02, J20 Conn_01x04, J21 Conn_01x04, J22 Conn_01x04, J23 Conn_01x06, J24 Conn_01x04, J25 Conn_01x02, J3 USB_C_Receptacle_USB2.0, J4 Micro_SD_Card, J5 Conn_01x06, J6 Conn_01x03, J7 Conn_01x03, J8 Conn_01x03, J9 Conn_01x03, Q1 TIP121, SW1 SW_Push, SW2 SW_Push, SW3 SW_DIP_x01, SW5 SW_SPDT, U1 CH32V203C8T6, U10 MPU-6050, U11 AMS1117-5.0, U12 AMS1117-3.3, U14 MCP4921-EMC, U2 CH32V203C8T6, U3 ADXL345BCCZ, U4 BMP280, U6 HMC5883L, U7 AMS1117-3.3, U8 PAM8403D, U9 AMS1117-5.0, Y1 8 MHZ, Y2 8 MHZ

Commit message: [ADD]: test code for PWM and ADC
Parts:
- removed SW5: SW_SPDT, Button_Switch_THT:SW_Slide_1P2T_CK_OS102011MS2Q
- added D5: 1N5819WS, Diode_SMD:D_SOD-323, F.Cu at (129.0, 107.6)
- added D6: 1N5819WS, Diode_SMD:D_SOD-323, F.Cu at (131.2, 110.2)
- added G***: LOGO, dummy:logo2, B.Cu at (88.3, 98.7)
- added G***: LOGO, dummy:logo2, B.Cu at (137.3, 98.6)
- added SW4: SW_SPDT, EG1218:SW_EG1218, F.Cu at (127.5, 102.7)
- J4: footprint Connector_Card:microSD_HC_Molex_47219-2001 -> footprints:J_SD_Card-micro_socket_A
- SW3: footprint Button_Switch_THT:SW_Slide_1P2T_CK_OS102011MS2Q -> EG1218:SW_EG1218
- moved SW3 2.62 mm to (97.4, 124.8)
- moved TP16 0.18 mm to (139.3, 59.7)
- moved H6 0.15 mm to (118.4, 68.2)
- turned J4 to 90 degrees
Routing:
- net GND_APPboard: track 436.8 -> 420.3 mm
- net /U2_PA6_ADC6: track 96.5 -> 85.2 mm
- net Net-(D6-K): track 38.9 -> 47.8 mm
- net /usb_vbus: track 56.6 -> 48.9 mm
- net Net-(D5-K): track 0.00 -> 6.06 mm
- net /U2_PC14_OSC32IN: track 83.6 -> 77.6 mm
- net /U2_PA5_ADC5: track 147.3 -> 141.8 mm, vias 11 -> 10
- net /U2_PC15_OSC32OUT: track 61.6 -> 56.8 mm, vias 3 -> 1
- net /U2_PA7_ADC7: track 122.3 -> 124.6 mm
- net /U2_PA1_ADC1: track 58.0 -> 59.2 mm
- net /U2_PA2_ADC2: track 22.9 -> 24.0 mm
- net /U2_PB4: track 92.2 -> 93.1 mm
- net /U2_PB3: track 125.2 -> 126.0 mm
- net /U2_PA9: track 92.9 -> 93.6 mm
- net Net-(U7-VI): track 23.8 -> 23.0 mm
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Other:
- board size 96.6 x 99.9 mm -> 96.6 x 100 mm
- board text added: "D0"
- board text added: "D1"
- board text added: "D2"
- board text added: "D3"
- board text added: "D4"
- board text added: "D5"
- board text added: "D6"
- board text added: "D7"
- board text added: "HREF"
- board text added: "MISO"
- board text added: "MOSI"
- board text added: "ON"
- board text added: "PCLK"
- board text added: "PWDN"
- board text added: "RESET"
- board text added: "SCK"
- board text added: "SCL"
- board text added: "SIOC"
- board text added: "SIOD"
- board text added: "USB_D+"
- board text added: "USB_D-"
- board text added: "VSYNC"
- board text added: "Version 1.0"
- board text added: "XCLK"
- board text added: "audio"
- board text added: "axdl_CS"
- board text added: "mcp_CS"
- board text added: "nrf_CS"
- board text added: "sd_CS"
- board text added: "uart_clk"
- board text added: "↑"

Commit message: [UPDATE]: create the skeleton project from the drone board
Parts:
- removed J3: USB_C_Receptacle_USB2.0, Connector_USB:USB_C_Receptacle_XKB_U262-16XN-4BVC11
- added J26: TYPE-C-31-M-12, TYPE-C-31-M-12:HRO_TYPE-C-31-M-12, F.Cu at (158.8, 131.4)
- D5, D6: footprint Diode_SMD:D_SOD-323 -> Diode_SMD:D_SMA
- U14: footprint Package_DFN_QFN:DFN-8-1EP_3x2mm_P0.5mm_EP1.75x1.45mm -> Package_SO:MSOP-8-1EP_3x3mm_P0.65mm_EP1.68x1.88mm
- moved D6 2.19 mm to (130.8, 112.4), turned to -90 degrees
- moved D5 0.85 mm to (129.4, 106.8)
- moved U14 0.67 mm to (147.9, 132.6)
- moved C6 0.32 mm to (82.8, 106.8)
Connections:
- J20 pad 3: /U1_PB14 -> /U1_PA1_ADC1
- J21 pad 3: /U1_PB12 -> /U1_PA11_USB1DM
- U3 pad 9: /U1_PA1_ADC1 -> /U1_PB14
- U6 pad 15: /U1_PA11_USB1DM -> /U1_PB12
Routing:
- net /U1_PA1_ADC1: track 37.3 -> 64.7 mm, vias 2 -> 3
- net /U1_PA11_USB1DM: track 52.9 -> 66.3 mm
- net /U2_PA5_ADC5: track 141.8 -> 149.3 mm
- net /U1_PB14: track 69.0 -> 76.0 mm, vias 4 -> 6
- net /U1_PB12: track 60.5 -> 65.9 mm, vias 4 -> 6
- net Net-(D6-K): track 47.8 -> 43.3 mm
- net /usb_vbus: track 48.9 -> 45.3 mm
- net 3.3V_APPboard: track 307.8 -> 310.3 mm
- net /U1_PB2_BOOT1: track 89.6 -> 87.4 mm
- net GND_Dboard: track 533.9 -> 535.9 mm
- net /U2_PB1_ADC9: track 87.4 -> 85.3 mm
- net /U2_PB2_BOOT1: track 139.2 -> 137.1 mm
- net 12V_APPboard: track 111.0 -> 109.1 mm, vias 7 -> 5
- net /U2_PB0_ADC8: track 83.6 -> 81.7 mm
- net /U1_PB4: track 122.2 -> 123.6 mm
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- added copper zone on F.Cu, net 3.3V_APPboard
- added copper zone on F.Cu, net 3.3V_Dboard
- added copper zone on B.Cu, net GND_APPboard
- added copper zone on B.Cu, net GND_Dboard
