File: hardware/pcb design files/quadraptor/quadraptor.kicad_sch (KiCad schematic)
At the start: 51 parts, among them J1 Conn_01x04, J2 Conn_01x02, J3 USB_C_Receptacle_USB2.0, J4 Micro_SD_Card, SW1 SW_Push, SW2 SW_Push, U1 CH32V203C8T6, U2 CH32V203C8T6, U3 ADXL345BCCZ, U4 BMP280, U5 MPU-6050_NRND, U6 HMC5883L, Y1 8 MHZ, Y2 8 MHZ

Commit message: [UPDATE]: initial schematic and pin assignments
Parts:
- added BZ1: Buzzer, symbol Device:Buzzer
- added C29, C30, C31, C32, C33: 10 uF, symbol Device:C
- added C34, C36, C37: 1 uF, symbol Device:C
- added C35: 470 uF, symbol Device:C
- added C38: 0.1 uF, symbol Device:C
- added C39, C40: 0.47 uF, symbol Device:C
- added D1, D2: LED, symbol Device:LED
- added H1, H2, H3, H4, H5, H6, H7, H8: MountingHole, symbol Mechanical:MountingHole
- added J10, J13, J5: Conn_01x04, symbol Connector_Generic:Conn_01x04
- added J11: Conn_02x09_Odd_Even, symbol Connector_Generic:Conn_02x09_Odd_Even
- added J12: Conn_02x04, 4ms_Connector:Pins_2x04_2.54mm_TH, symbol PCM_4ms_Connector:Conn_02x04
- added J14, J15, J16, J17, J18: Conn_01x02, symbol Connector_Generic:Conn_01x02
- added J6, J7, J8, J9: Conn_01x03, symbol Connector_Generic:Conn_01x03
- added LS1, LS2: Speaker (3W 4ohm), symbol Device:Speaker
- added Q1: TIP121, Package_TO_SOT_THT_AKL:TO-220-3_Vertical_BCE, symbol PCM_Transistor_BJT_Darlington_AKL:TIP121
- added R10, R9: 10 Kohm, symbol Device:R
- added R11, R12: 20 Kohm, symbol Device:R
- added R13: 1 Kohm, symbol Device:R
- added R3: 15 Kohm, symbol Device:R
- added R4: 4.7 Kohm, symbol Device:R
- added R5, R8: 330 ohm, symbol Device:R
- added R6, R7: 5.1 Kohm, symbol Device:R
- added SW3: SW_DIP_x01, symbol Switch:SW_DIP_x01
- added SW5: SW_DPDT_x2, symbol Switch:SW_DPDT_x2
- added TP10, TP11, TP12, TP13, TP14, TP15, TP16, TP17, TP18, TP19, TP20, TP21, TP22, TP23, TP8, TP9: TestPoint, symbol Connector:TestPoint
- added U10, U7: LD1117S33CTR, digikey-footprints:SOT-223, symbol dk_PMIC-Voltage-Regulators-Linear:LD1117S33CTR
- added U11: AMS1117-5.0, Package_TO_SOT_SMD:SOT-223-3_TabPin2, symbol Regulator_Linear:AMS1117-5.0
- added U13: 74HC165, symbol 74xx:74HC165
- added U14: MCP4921-EMC, Package_DFN_QFN:DFN-8-1EP_3x2mm_P0.5mm_EP1.75x1.45mm, symbol Analog_DAC:MCP4921-EMC
- added U8: PAM8403D, Package_SO:SOP-16_3.9x9.9mm_P1.27mm, symbol Amplifier_Audio:PAM8403D
- R1, R2: value R -> 4.7 Kohm
Connections:
- net adxl345_INT1 is gone; now on net U1_PA9: U3.8 (INT1)
- net adxl345_INT2 is gone; now on net U1_PA10: U3.9 (INT2)
- net hmc5883_DRDY is gone; now on net U1_PA11_USB1DM: U6.15 (DRDY)
- net mpu6050_INT is gone; now on net U1_PA12_USB1DP: U5.12 (INT)
- net +3.3V: now also C9.1, J4.4 (VDD), C31.1, D1.2 (A), D2.2 (A), J11.1 (Pin_1), J11.17 (Pin_17), J12.2 (Pin_2), J13.1 (Pin_1), R10.1, R9.1, TP22.1, TP23.1, U10.2 (VOUT), U10.4 (VOUT), U13.16 (VCC), U14.1 (Vdd), U14.6 (Vref), U7.2 (VOUT), U7.4 (VOUT); no longer J2.1 (Pin_1)
- net GND: now also C9.2, J3.A1 (GND), J3.A12 (GND), J3.B1 (GND), J3.B12 (GND), J3.S1 (SHIELD), J4.6 (VSS), J4.9 (SHIELD), BZ1.2 (+), C29.2, C30.2, C31.2, C32.2, C33.2, C34.2, C35.2, C36.2, C37.2, C38.2, J10.4 (Pin_4), J11.18 (Pin_18), J11.2 (Pin_2), J12.1 (Pin_1), J13.4 (Pin_4), J14.2 (Pin_2), J5.4 (Pin_4), J6.3 (Pin_3), J7.3 (Pin_3), J8.3 (Pin_3), J9.3 (Pin_3), Q1.3 (E), R4.2, R5.1, R6.2, R7.2, R8.1, U10.1 (GND), U11.1 (GND), U13.8 (GND), U14.5 (~{LDAC}), U14.7 (Vss), U14.9 (PAD/Vss), U7.1 (GND), U8.11 (GND), U8.15 (PGND), U8.2 (PGND)
- net U1_PA4_ADC4: now also R3.2, R4.1
- net U1_PB0_ADC8: now also J5.1 (Pin_1)
- net U1_PB1_ADC9: now also J5.2 (Pin_2)
- net U1_PB2_BOOT1: now also J5.3 (Pin_3)
- net U1_PB6_USB2DM: now also J9.1 (Pin_1)
- net U1_PB7_USB2DP: now also J8.1 (Pin_1)
- net U1_PB8: now also J6.1 (Pin_1)
- net U1_PB9: now also J7.1 (Pin_1)
- net U2_PA0_WKUP_ADC0: now also TP16.1, U13.1 (~{PL})
- net U2_PA10: now also TP19.1, U14.2 (~{CS})
- net U2_PA11_USB1DM: now also J11.6 (Pin_6)
- net U2_PA12_USB1DP: now also J11.5 (Pin_5)
- net U2_PA13_SWDIO: now also J13.2 (Pin_2)
- net U2_PA14_SWCLK: now also J13.3 (Pin_3)
- net U2_PA15: now also J11.7 (Pin_7)
- net U2_PA1_ADC1: now also BZ1.1 (-)
- net U2_PA5_ADC5: now also J4.5 (CLK), J12.5 (Pin_5), TP8.1, U14.3 (SCK)
- net U2_PA6_ADC6: now also J4.7 (DAT0), J12.7 (Pin_7), TP9.1
- net U2_PA7_ADC7: now also J4.3 (CMD), J12.6 (Pin_6), TP10.1, U14.4 (SDI)
- net U2_PA8: now also J11.8 (Pin_8)
- net U2_PA9: now also TP15.1, U13.9 (Q7)
- net U2_PB0_ADC8: now also J10.2 (Pin_2)
- net U2_PB10: now also J11.3 (Pin_3), R9.2, TP13.1
- net U2_PB11: now also J11.4 (Pin_4), R10.2, TP14.1
- net U2_PB15: now also J12.8 (Pin_8)
- net U2_PB1_ADC9: now also J10.1 (Pin_1)
- net U2_PB2_BOOT1: now also J10.3 (Pin_3)
- net U2_PB5: now also TP17.1, U13.15 (~{CE})
- net U2_PB6_USB2DM: now also J3.A7 (D-), J3.B7 (D-)
- net U2_PB7_USB2DP: now also J3.A6 (D+), J3.B6 (D+)
- net U2_PB8: now also TP18.1, U13.2 (CP)
- net U2_PB9: now also R13.2
- net U2_PC14_OSC32IN: now also J12.3 (Pin_3), TP11.1
- net U2_PC15_OSC32OUT: now also J4.2 (DAT3/CD), TP12.1
- net usb_vbus: now reaches J3.A4 (VBUS), J3.A9 (VBUS), J3.B4 (VBUS), J3.B9 (VBUS)
- net usb_vbus: now also SW5.4 (A)
- net at J3.A5 (CC1): now also R6.1
- net at J3.B5 (CC2): now also R7.1
- new net: C29.1, SW3.2, U7.3 (VIN)
- new net: D1.1 (K), R5.2
- new net: C39.1, C40.1, TP21.1, U14.8 (Vout)
- new net: C40.2, R12.2
- new net: Q1.1 (B), R13.1
- new net: R12.1, U8.10 (INR)
- new net: LS2.1, U8.14 (ROUT-)
- new net: LS2.2, U8.16 (ROUT+)
- new net: D2.1 (K), R8.2
- new net: C30.1, SW5.5 (B), U10.3 (VIN)
- new net: LS1.1, U8.1 (LOUT+)
- new net: LS1.2, U8.3 (LOUT-)
- new net: J15.2 (Pin_2), J16.2 (Pin_2), J17.2 (Pin_2), J18.2 (Pin_2), Q1.2 (C)
- new net: R11.1, U8.7 (INL)
- new net: C39.2, R11.2
- new net: C38.1, U8.8 (VREF)
- new net +12V: C32.1, J14.1 (Pin_1), J15.1 (Pin_1), J16.1 (Pin_1), J17.1 (Pin_1), J18.1 (Pin_1), J2.1 (Pin_1), R3.1, SW3.1, SW5.6 (C), U11.3 (VI)
- new net +5V: C33.1, C34.1, C35.1, C36.1, C37.1, TP20.1, U11.2 (VO), U8.12 (~{SHDN}), U8.13 (PVDD), U8.4 (PVDD), U8.5 (~{MUTE}), U8.6 (VDD)
- new net camera_D0: J11.16 (Pin_16), U13.11 (D0)
- new net camera_D1: J11.15 (Pin_15), U13.12 (D1)
- new net camera_D2: J11.14 (Pin_14), U13.13 (D2)
- new net camera_D3: J11.13 (Pin_13), U13.14 (D3)
- new net camera_D4: J11.12 (Pin_12), U13.3 (D4)
- new net camera_D5: J11.11 (Pin_11), U13.4 (D5)
- new net camera_D6: J11.10 (Pin_10), U13.5 (D6)
- new net camera_D7: J11.9 (Pin_9), U13.6 (D7)
- no-connect marks 4 -> 38
Other:
- note added: "74HC165 (p-in, s-out)"
- note added: "Address = 0x1E"
- note added: "Address = 0x68"
- note added: "Audio"
- note added: "CE"
- note added: "CNS"
- note added: "Clk"
- note added: "D0"
- note added: "D1"
- note added: "D2"
- note added: "D3"
- note added: "D4"
- note added: "D5"
- note added: "D6"
- note added: "D7"
- note added: "HREF"
- note added: "IRQ"
- note added: "LED control"
- note added: "MISO"
- note added: "MOSI"
- note added: "Motor interface with ESCs"
- note added: "PCLK"
- note added: "PWDN"
- note added: "Pin Headers & interfaces"
- note added: "Power"
- note added: "RESET"
- note added: "SCK"
- note added: "SCL"
- note added: "SDA"
- note added: "SPI interface with wireless receiver"
- note added: "UART interface with application board"
- note added: "UART interface with drone board"
- note added: "VSYNK"
- note added: "XCLK"
- note added: "battery monitor"
- note added: "camera interface"
- note added: "clk enable"
- note added: "fast mode of I2C is used"
- note added: "serial in"
- note added: "shift/load"
- moved on the sheet: C9, J1, J2, J3, J4, R1, R2, TP1, TP2, TP3, TP4, TP5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

Commit message: [UPDATE]: complete initial code for the remote control
Parts:
- added J19, J20, J21, J22: Conn_01x04, symbol Connector_Generic:Conn_01x04
- added J5: Conn_01x06, symbol Connector_Generic:Conn_01x06
- J?: renamed from J5; value Conn_01x04 -> Conn_01x06; symbol Connector_Generic:Conn_01x04 -> Connector_Generic:Conn_01x06
- U1, U2: footprint (none) -> CH32V203:CH32V203C8T6_LQFP-48_7x7mm_P0.5mm
Connections:
- net +3.3V: now also J10.1 (Pin_1), J19.1 (Pin_1), J20.1 (Pin_1), J21.1 (Pin_1), J22.1 (Pin_1)
- net GND: now also J?.6 (Pin_6), J19.4 (Pin_4), J20.4 (Pin_4), J21.4 (Pin_4), J22.4 (Pin_4), J5.6 (Pin_6); no longer J?.4 (Pin_4)
- net U1_PA15: now also J22.3 (Pin_3)
- net U1_PA2_ADC2: now also J10.3 (Pin_3)
- net U1_PA3_ADC3: now also J19.3 (Pin_3)
- net U1_PA8: now also J22.2 (Pin_2)
- net U1_PB12: now also J21.3 (Pin_3)
- net U1_PB13: now also J20.2 (Pin_2)
- net U1_PB14: now also J20.3 (Pin_3)
- net U1_PB15: now also J19.2 (Pin_2)
- net U1_PB3: now also J?.4 (Pin_4)
- net U1_PB4: now also J?.5 (Pin_5)
- net U1_PB5: now also J21.2 (Pin_2)
- net U1_PC13_TAMPER_RTC: now also J10.2 (Pin_2)
- net U2_PB0_ADC8: now also J5.2 (Pin_2); no longer J10.2 (Pin_2)
- net U2_PB1_ADC9: now also J5.1 (Pin_1); no longer J10.1 (Pin_1)
- net U2_PB2_BOOT1: now also J5.3 (Pin_3); no longer J10.3 (Pin_3)
- net U2_PB3: now also J5.5 (Pin_5)
- net U2_PB4: now also J5.4 (Pin_4)
- net U2_PC13_TAMPER_RTC: now also J12.4 (Pin_4)
- no-connect marks 38 -> 25
Other:
- note added: "CK"
- note added: "CTS"
- note added: "Echo"
- note added: "RTS"
- note added: "RX"
- note added: "TX"
- note added: "Trig"
- note added: "Ultrasound sensors"
- note added: "max speed = 10Mbps"
- moved on the sheet: H1, H2, H3, H4, J1, J13, J14, J2, J6, J7, J8, J9

Commit message: [UPDATE]: completed initial PCB routing and design
Parts:
- removed C17, C18, C19, C26: 0.1 uF, symbol Device:C
- removed C20: 220 pF, symbol Device:C
- removed SW5: SW_DPDT_x2, symbol Switch:SW_DPDT_x2
- removed TP18, TP20, TP22: TestPoint, symbol Connector:TestPoint
- removed U10, U7: LD1117S33CTR, digikey-footprints:SOT-223, symbol dk_PMIC-Voltage-Regulators-Linear:LD1117S33CTR
- removed U13: 74HC165, symbol 74xx:74HC165
- removed U5: MPU-6050_NRND, digikey-footprints:QFN-24-1EP_4x4mm, symbol dk_Motion-Sensors-IMUs-Inertial-Measurement-Units:MPU-6050_NRND
- added C41, C42: 10 uF, Capacitor_SMD:C_1206_3216Metric_Pad1.33x1.80mm_HandSolder, symbol Device:C
- added C43, C44, C45, C46, C47: 0.1 uF, Capacitor_SMD:C_0805_2012Metric_Pad1.18x1.45mm_HandSolder, symbol Device:C
- added D3, D4: LED, LED_SMD:LED_0805_2012Metric_Pad1.15x1.40mm_HandSolder, symbol Device:LED
- added J24: Conn_01x04, Connector_JST:JST_XH_B4B-XH-A_1x04_P2.50mm_Vertical, symbol Connector_Generic:Conn_01x04
- added J25: Conn_01x02, Connector_PinHeader_2.54mm:PinHeader_1x02_P2.54mm_Vertical, symbol Connector_Generic:Conn_01x02
- added R14, R18: 10Kohm, Resistor_SMD:R_0805_2012Metric_Pad1.20x1.40mm_HandSolder, symbol Device:R
- added R15, R19: 10 Kohm, Resistor_SMD:R_0805_2012Metric_Pad1.20x1.40mm_HandSolder, symbol Device:R
- added R16, R17: 330 ohm, Resistor_SMD:R_0603_1608Metric_Pad0.98x0.95mm_HandSolder, symbol Device:R
- added SW5: SW_SPDT, Button_Switch_THT:SW_Slide_1P2T_CK_OS102011MS2Q, symbol Switch:SW_SPDT
- added TP24, TP25, TP27, TP28: TestPoint, TestPoint:TestPoint_Bridge_Pitch2.54mm_Drill1.0mm, symbol Connector:TestPoint
- added U10: MPU-6050, Sensor_Motion:InvenSense_QFN-24_4x4mm_P0.5mm, symbol Sensor_Motion:MPU-6050
- added U12, U7: AMS1117-3.3, Package_TO_SOT_SMD:SOT-223-3_TabPin2, symbol Regulator_Linear:AMS1117-3.3
- added U9: AMS1117-5.0, Package_TO_SOT_SMD:SOT-223-3_TabPin2, symbol Regulator_Linear:AMS1117-5.0
- BZ1: footprint (none) -> Buzzer_Beeper:Buzzer_12x9.5RM7.6
- C1, C21, C22, C23, C25, C4: value 0.1 uF -> 0.1uF; footprint (none) -> Capacitor_SMD:C_0805_2012Metric_Pad1.18x1.45mm_HandSolder
- C10, C11, C12, C14, C15, C16, C2, C24, C27, C28, C34, C36, C37, C38, C39, C40, C5, C6, C7, C8: footprint (none) -> Capacitor_SMD:C_0805_2012Metric_Pad1.18x1.45mm_HandSolder
- C13, C29, C30, C31, C32, C33, C9: footprint (none) -> Capacitor_SMD:C_1206_3216Metric_Pad1.33x1.80mm_HandSolder
- C3: value 0.1 uF -> 220 pF; footprint (none) -> Capacitor_SMD:C_0805_2012Metric_Pad1.18x1.45mm_HandSolder
- C35: footprint (none) -> Capacitor_THT:CP_Radial_D5.0mm_P2.00mm
- D1, D2: footprint (none) -> LED_SMD:LED_0805_2012Metric_Pad1.15x1.40mm_HandSolder
- H1, H2, H3, H4, H5, H6, H7, H8: footprint (none) -> MountingHole:MountingHole_3.2mm_M3
- J1, J13: footprint (none) -> Connector_PinHeader_2.54mm:PinHeader_1x04_P2.54mm_Vertical
- J10, J19, J20, J21, J22: footprint (none) -> Connector_PinSocket_2.54mm:PinSocket_1x04_P2.54mm_Vertical
- J11: footprint (none) -> Connector_PinHeader_2.54mm:PinHeader_2x09_P2.54mm_Vertical
- J12: footprint 4ms_Connector:Pins_2x04_2.54mm_TH -> Connector_PinHeader_2.54mm:PinHeader_2x04_P2.54mm_Vertical
- J14, J15, J16, J17, J18, J2: footprint (none) -> Connector_JST:JST_XH_B2B-XH-A_1x02_P2.50mm_Vertical
- J23: renamed from J?; footprint (none) -> Connector_JST:JST_XH_B6B-XH-A_1x06_P2.50mm_Vertical
- J3: footprint (none) -> Connector_USB:USB_C_Receptacle_XKB_U262-16XN-4BVC11
- J4: footprint (none) -> Connector_Card:microSD_HC_Molex_47219-2001
- J5: footprint (none) -> Connector_JST:JST_XH_B6B-XH-A_1x06_P2.50mm_Vertical
- J6, J7, J8, J9: footprint (none) -> Connector_PinHeader_2.54mm:PinHeader_1x03_P2.54mm_Vertical
- LS1, LS2: footprint (none) -> Connector_PinHeader_2.54mm:PinHeader_1x02_P2.54mm_Vertical
- Q1: footprint Package_TO_SOT_THT_AKL:TO-220-3_Vertical_BCE -> Package_TO_SOT_THT:TO-220-3_Vertical
- R1, R10, R11, R12, R13, R2, R3, R4, R6, R7, R9: footprint (none) -> Resistor_SMD:R_0805_2012Metric_Pad1.20x1.40mm_HandSolder
- R5, R8: footprint (none) -> Resistor_SMD:R_0603_1608Metric_Pad0.98x0.95mm_HandSolder
- SW1, SW2: footprint (none) -> Button_Switch_SMD:SW_Push_1P1T_NO_6x6mm_H9.5mm
- SW3: footprint (none) -> Button_Switch_THT:SW_Slide_1P2T_CK_OS102011MS2Q
- TP1, TP10, TP11, TP12, TP13, TP14, TP15, TP16, TP17, TP19, TP2, TP21, TP23, TP3, TP4, TP5, TP6, TP7, TP8, TP9: footprint (none) -> TestPoint:TestPoint_Bridge_Pitch2.54mm_Drill1.0mm
- Y1, Y2: footprint (none) -> Crystal:Crystal_HC18-U_Vertical
Connections:
- net camera_D0 is gone; now on net U2_PA0_WKUP_ADC0: J11.16 (Pin_16)
- net camera_D1 is gone; now on net U2_PB8: J11.15 (Pin_15)
- net camera_D2 is gone; now on net U2_PB5: J11.14 (Pin_14)
- net camera_D3 is gone; now on net U2_PA9: J11.13 (Pin_13)
- net camera_D4 is gone; now on net U2_PB14: J11.12 (Pin_12)
- net camera_D5 is gone; now on net U2_PB13: J11.11 (Pin_11)
- net camera_D6 is gone; now on net U2_PB12: J11.10 (Pin_10)
- net camera_D7 is gone; now on net U2_PA4_ADC4: J11.9 (Pin_9)
- net U1_NRST: now also R14.2
- net U1_PA0_WKUP_ADC0: now also U3.8 (INT1)
- net U1_PA10: now also J24.3 (Pin_3); no longer U3.9 (INT2)
- net U1_PA12_USB1DP: now also U10.12 (INT)
- net U1_PA1_ADC1: now also U3.9 (INT2)
- net U1_PA9: now also J24.2 (Pin_2); no longer U3.8 (INT1)
- net U1_PB0_ADC8: now also TP27.1
- net U1_PB10: now also U10.23 (SCL)
- net U1_PB11: now also U10.24 (SDA)
- net U1_PB1_ADC9: now also TP28.1
- net U2_NRST: now also R15.2
- net U2_PA0_WKUP_ADC0: no longer TP16.1
- net U2_PA2_ADC2: now also J25.1 (Pin_1)
- net U2_PA3_ADC3: now also J25.2 (Pin_2)
- net U2_PA9: no longer TP15.1
- net U2_PB2_BOOT1: now also TP17.1
- net U2_PB5: no longer TP17.1
- net U2_PB6_USB2DM: now also TP15.1
- net U2_PB7_USB2DP: now also TP16.1
- net hmc5883_SCL: now also U10.7 (AUX_CL)
- net hmc5883_SDA: now also U10.6 (AUX_DA)
- net usb_vbus: now also SW5.1 (A)
- net at C29.1, SW3.2: now also U7.3 (VI)
- net at C30.1: now also SW5.2 (B), U12.3 (VI)
- net +12V renamed 12V_APPboard
- net 12V_APPboard: now also SW5.3 (C); no longer J2.1 (Pin_1), R3.1, SW3.1
- net +3.3V renamed 3.3V_Dboard
- net 3.3V_Dboard: now also J24.1 (Pin_1), R14.1, U10.13 (VDD), U10.8 (VLOGIC), U7.2 (VO); no longer C3.1, C31.1, C6.1, D2.2 (A), J10.1 (Pin_1), J11.1 (Pin_1), J11.17 (Pin_17), J12.2 (Pin_2), J13.1 (Pin_1), J19.1 (Pin_1), J20.1 (Pin_1), J21.1 (Pin_1), J22.1 (Pin_1), J4.4 (VDD), R10.1, R9.1, U14.1 (Vdd), U14.6 (Vref), U2.1 (VBAT), U2.24 (VDD_VIO1), U2.36 (VDD_2), U2.48 (VDD_VIO_3), U2.9 (VDDA)
- net +5V renamed 5V_APPboard
- net 5V_APPboard: now also D4.2 (A)
- net GND renamed GND_Dboard
- net GND_Dboard: now also C41.2, C42.2, J24.4 (Pin_4), R16.1, R18.2, TP25.1, U10.1 (CLKIN), U10.11 (FSYNC), U10.18 (GND), U10.9 (AD0), U7.1 (GND), U9.1 (GND); no longer BZ1.2 (+), C24.2, C27.2, C28.2, C30.2, C31.2, C32.2, C33.2, C34.2, C35.2, C36.2, C37.2, C38.2, J11.18 (Pin_18), J11.2 (Pin_2), J12.1 (Pin_1), J13.4 (Pin_4), J14.2 (Pin_2), J3.A1 (GND), J3.A12 (GND), J3.B1 (GND), J3.B12 (GND), J3.S1 (SHIELD), J4.6 (VSS), J4.9 (SHIELD), J5.6 (Pin_6), Q1.3 (E), R6.2, R7.2, R8.1, SW2.1, U1.44 (BOOT0), U11.1 (GND), U14.5 (~{LDAC}), U14.7 (Vss), U14.9 (PAD/Vss), U2.23 (VSS1), U2.35 (VSS_2), U2.44 (BOOT0), U2.47 (VSS_3), U2.8 (VSSA), U8.11 (GND), U8.15 (PGND), U8.2 (PGND)
- new net: C6.1, U10.10 (REGOUT)
- new net: C3.1, U10.20 (CPOUT)
- new net: D4.1 (K), R17.2
- new net: D3.1 (K), R16.2
- new net 12V_Dboard: C41.1, J2.1 (Pin_1), R3.1, SW3.1, U9.3 (VI)
- new net 3.3V_APPboard: C31.1, C43.1, C44.1, C45.2, C46.2, C47.1, D2.2 (A), J11.1 (Pin_1), J11.17 (Pin_17), J12.2 (Pin_2), J13.1 (Pin_1), J4.4 (VDD), R10.1, R15.1, R9.1, U12.2 (VO), U14.1 (Vdd), U14.6 (Vref), U2.1 (VBAT), U2.24 (VDD_VIO1), U2.36 (VDD_2), U2.48 (VDD_VIO_3), U2.9 (VDDA)
- new net 5V_Dboard: C42.1, D3.2 (A), J10.1 (Pin_1), J19.1 (Pin_1), J20.1 (Pin_1), J21.1 (Pin_1), J22.1 (Pin_1), TP24.1, U9.2 (VO)
- new net GND_APPboard: BZ1.2 (+), C24.2, C27.2, C28.2, C30.2, C31.2, C32.2, C33.2, C34.2, C35.2, C36.2, C37.2, C38.2, C43.2, C44.2, C45.1, C46.1, C47.2, J11.18 (Pin_18), J11.2 (Pin_2), J12.1 (Pin_1), J13.4 (Pin_4), J14.2 (Pin_2), J3.A1 (GND), J3.A12 (GND), J3.B1 (GND), J3.B12 (GND), J3.S1 (SHIELD), J4.6 (VSS), J4.9 (SHIELD), J5.6 (Pin_6), Q1.3 (E), R17.1, R19.2, R6.2, R7.2, R8.1, SW2.1, U11.1 (GND), U12.1 (GND), U14.5 (~{LDAC}), U14.7 (Vss), U14.9 (PAD/Vss), U2.23 (VSS1), U2.35 (VSS_2), U2.47 (VSS_3), U2.8 (VSSA), U8.11 (GND), U8.15 (PGND), U8.2 (PGND)
- new net U1_BOOT0: R18.1, U1.44 (BOOT0)
- new net U2_BOOT0: R19.1, U2.44 (BOOT0)
- no-connect marks 25 -> 10
Other:
- note added: "CS"
- note added: "GPS interface"
- note added: "unconnected pins"
- note removed: "74HC165 (p-in, s-out)"
- note removed: "Clk"
- note removed: "clk enable"
- note removed: "serial in"
- note removed: "shift/load"
- moved on the sheet: BZ1, C11, C12, C24, C27, C28, C29, C34, C35, C36, C37, C38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

Commit message: [ADD]: test code for PWM and ADC
Parts:
- removed SW5: SW_SPDT, Button_Switch_THT:SW_Slide_1P2T_CK_OS102011MS2Q, symbol Switch:SW_SPDT
- added D5, D6: 1N5819WS, Diode_SMD:D_SOD-323, symbol Diode:1N5819WS
- added SW4: SW_SPDT, EG1218:SW_EG1218, symbol Switch:SW_SPDT
- J4: footprint Connector_Card:microSD_HC_Molex_47219-2001 -> footprints:J_SD_Card-micro_socket_A
- SW3: footprint Button_Switch_THT:SW_Slide_1P2T_CK_OS102011MS2Q -> EG1218:SW_EG1218
Connections:
- net 12V_APPboard: now also D5.2 (A)
- net usb_vbus: now also D6.2 (A)
- net at C30.1, U12.3 (VI): now also D6.1 (K), SW4.2 (B)
- new net: D5.1 (K), SW4.1 (A)
- no-connect marks 10 -> 11
Other:
- note added: "ADXL_CS"
- note added: "BMP280_CS"
- note added: "mcp_CS"
- note added: "nrf_CS"
- note added: "sd_CS"
